File: Project-1-LED-Torch/Project-1-LED-Torch.kicad_sch (KiCad schematic)
At the start: 4 parts, among them SW1 SW_DPDT_x2

Commit message: do schematic design, step 7, add comments inc footprints notes
Other:
- note added: "A simple LED Torch circuit"
Changed lines of the file:
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@@
 		(company "Jupiter SW")
+	)
+	(rectangle
+		(start 87.63 66.04)
+		(end 194.945 102.235)
+		(stroke
+			(width 0)
+			(type default)
+		)
+		(fill
+			(type none)
+		)
+	)
+	(text "A simple LED Torch circuit"
+		(exclude_from_sim no)
+		(at 100.33 64.77 0)
+		(effects
+			(font
+				(size 1.27 1.27)
+			)
+			(href "https://jupitersw.com")
+		)
 	)
 	(wire
@@
 		(in_pos_files yes)
 		(dnp no)
-		(fields_autoplaced yes)
 		(property "Reference" "R1"
 			(at 130.81 69.85 90)
@@
 		)
 		(property "Footprint" "Resistor_THT:R_Axial_DIN0204_L3.6mm_D1.6mm_P7.62mm_Horizontal"
-			(at 130.81 77.978 90)
-			(hide yes)
+			(at 160.655 81.915 90)
 			(show_name no)
 			(do_not_autoplace no)
@@
 		(in_pos_files yes)
 		(dnp no)
-		(fields_autoplaced yes)
 		(property "Reference" "D1"
 			(at 107.6325 69.85 0)
@@
 		)
 		(property "Footprint" "LED_THT:LED_D5.0mm"
-			(at 109.22 76.2 0)
-			(hide yes)
+			(at 112.395 80.645 0)
 			(show_name no)
 			(do_not_autoplace no)
@@
 		(in_pos_files yes)
 		(dnp no)
-		(fields_autoplaced yes)
 		(property "Reference" "SW1"
 			(at 148.59 69.85 0)
@@
 		)
 		(property "Footprint" "Button_Switch_THT:SW_TH_Tactile_Omron_B3F-100x"
-			(at 148.59 76.2 0)
-			(hide yes)
+			(at 167.64 78.105 0)
 			(show_name no)
 			(do_not_autoplace no)
@@
 		(in_pos_files yes)
 		(dnp no)
-		(fields_autoplaced yes)
 		(property "Reference" "BT1"
 			(at 132.6515 87.63 90)
@@
 		)
 		(property "Footprint" "Battery:BatteryHolder_Keystone_1058_1x2032"
-			(at 132.334 95.25 90)
-			(hide yes)
-			(show_name no)
-			(do_not_autoplace no)
+			(at 130.81 99.06 90)
+			(show_name no)
+			(do_not_autoplace no)

Commit message: do schematic design, step 7, add comments inc footprints notes
Other:
- note added: "A simple LED Torch circuit, using a coin cell battery holder."
- note removed: "A simple LED Torch circuit"
Changed lines of the file:
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@@
 		)
 	)
-	(text "A simple LED Torch circuit"
-		(exclude_from_sim no)
-		(at 100.33 64.77 0)
+	(text "A simple LED Torch circuit, using a coin cell battery holder."
+		(exclude_from_sim no)
+		(at 117.475 64.77 0)
 		(effects
 			(font
@@
 		)
 		(property "Footprint" "Resistor_THT:R_Axial_DIN0204_L3.6mm_D1.6mm_P7.62mm_Horizontal"
-			(at 160.655 81.915 90)
-			(show_name no)
-			(do_not_autoplace no)
-			(effects
-				(font
-					(size 1.27 1.27)
+			(at 131.445 78.74 90)
+			(show_name no)
+			(do_not_autoplace no)
+			(effects
+				(font
+					(size 0.5 0.5)
 				)
 			)
@@
 		)
 		(property "Footprint" "LED_THT:LED_D5.0mm"
-			(at 112.395 80.645 0)
-			(show_name no)
-			(do_not_autoplace no)
-			(effects
-				(font
-					(size 1.27 1.27)
+			(at 109.22 80.01 0)
+			(show_name no)
+			(do_not_autoplace no)
+			(effects
+				(font
+					(size 0.5 0.5)
 				)
 			)
@@
 		)
 		(property "Footprint" "Button_Switch_THT:SW_TH_Tactile_Omron_B3F-100x"
-			(at 167.64 78.105 0)
-			(show_name no)
-			(do_not_autoplace no)
-			(effects
-				(font
-					(size 1.27 1.27)
+			(at 148.59 77.47 0)
+			(show_name no)
+			(do_not_autoplace no)
+			(effects
+				(font
+					(size 0.5 0.5)
 				)
 			)
@@
 			(effects
 				(font
-					(size 1.27 1.27)
-				)
-			)
+					(size 0.5 0.5)
+				)
+			)

Commit message: do PCB layout design, step 8, setup
Changed lines of the file:
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@@
 	(rectangle
 		(start 87.63 66.04)
-		(end 194.945 102.235)
+		(end 170.18 102.235)
 		(stroke
 			(width 0)
