File: Project-2-Breadboard-Power-Supply/Project-2-Breadboard-Power-Supply.kicad_pcb (KiCad board)
At the start: 2 copper layers, 33.2 x 52.5 mm, 18 parts, among them J1 Conn_01x02_Pin, J2 Conn_01x02_Pin, J3 Conn_01x03_Pin, J4 Conn_01x03_Pin, J5 Screw_Terminal_01x02, J6 Barrel_Jack_Switch, J7 Screw_Terminal_01x02, U1 LM7805_TO220, U2 LM317_TO-220

Commit message: update front and back silkscreen footprints and free text to clear warnings
Parts:
- moved REF** 19.8 mm to (33.0, 71.5)
Other:
- board text added: "v0.1"
- board text removed: "version0.1"
Changed lines of the file:
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@@
 			(effects
 				(font
-					(size 0.7 0.7)
+					(size 0.8 0.8)
 					(thickness 0.15)
 				)
@@
 			(effects
 				(font
-					(size 0.7 0.7)
+					(size 0.8 0.8)
 					(thickness 0.15)
 				)
@@
 			(effects
 				(font
-					(size 0.7 0.7)
+					(size 0.7 0.8)
 					(thickness 0.108)
 				)
@@
 			(effects
 				(font
-					(size 0.7 0.7)
+					(size 0.8 0.8)
 					(thickness 0.15)
 				)
@@
 			(effects
 				(font
-					(size 0.7 0.7)
+					(size 0.8 0.8)
 					(thickness 0.15)
 				)
@@
 			(effects
 				(font
-					(size 0.7 0.7)
+					(size 0.7 0.8)
 					(thickness 0.15)
 				)
@@
 			(effects
 				(font
-					(size 0.7 0.7)
+					(size 0.8 0.8)
 					(thickness 0.15)
 				)
@@
 			(effects
 				(font
-					(size 0.7 0.7)
+					(size 0.8 0.8)
 					(thickness 0.15)
 				)
@@
 			(effects
 				(font
-					(size 0.7 0.7)
+					(size 0.8 0.8)
 					(thickness 0.15)
 				)
@@
 			(effects
 				(font
-					(size 0.7 0.7)
+					(size 0.8 0.8)
 					(thickness 0.15)
 				)
@@
 			(effects
 				(font
-					(size 0.7 0.7)
+					(size 0.8 0.8)
 					(thickness 0.15)
 				)
@@
 			(effects
 				(font
-					(size 0.7 0.7)
+					(size 0.7 0.8)
 					(thickness 0.15)
 				)
@@
 			(effects
 				(font
-					(size 0.7 0.7)
+					(size 0.8 0.8)
 					(thickness 0.15)
 				)
@@
 			(effects
 				(font
-					(size 0.7 0.7)
+					(size 0.8 0.8)
 					(thickness 0.15)
 				)
@@
 			(effects
 				(font
-					(size 0.7 0.7)
+					(size 0.7 0.8)
 					(thickness 0.09)
 				)
@@
 			(effects
 				(font
-					(size 0.7 0.7)
+					(size 0.8 0.8)
 					(thickness 0.15)
 				)
@@
 			(effects
 				(font
-					(size 0.7 0.7)
+					(size 0.8 0.8)
 					(thickness 0.15)
 				)
@@
 			(effects
 				(font
-					(size 0.7 0.7)
+					(size 0.7 0.8)
 					(thickness 0.12)
 				)
@@
 			(effects
 				(font
-					(size 0.7 0.7)
+					(size 0.8 0.8)
 					(thickness 0.15)
 				)
@@
 			(effects
 				(font
-					(size 0.7 0.7)
+					(size 0.8 0.8)
 					(thickness 0.15)
 				)
@@
 			(effects
 				(font
-					(size 0.7 0.7)
+					(size 0.7 0.8)
 					(thickness 0.15)
 				)
@@
 			(effects
 				(font
-					(size 0.7 0.7)
+					(size 0.8 0.8)
 					(thickness 0.15)
 				)
@@
 			(effects
 				(font
-					(size 0.7 0.7)
+					(size 0.8 0.8)
 					(thickness 0.15)
 				)
@@
 			(effects
 				(font
-					(size 0.7 0.7)
+					(size 0.7 0.8)
 					(thickness 0.15)
 				)
@@
 			(effects
 				(font
-					(size 0.7 0.7)
+					(size 0.8 0.8)
 					(thickness 0.15)
 				)
@@
 			(effects
 				(font
-					(size 0.7 0.7)
+					(size 0.8 0.8)
 					(thickness 0.15)
 				)
@@
 			(effects
 				(font
-					(size 0.7 0.7)
+					(size 0.7 0.8)
 					(thickness 0.108)
 				)
@@
 			(effects
 				(font
-					(size 0.7 0.7)
+					(size 0.8 0.8)
 					(thickness 0.15)
 				)
@@
 			(effects
 				(font
-					(size 0.7 0.7)
+					(size 0.8 0.8)
 					(thickness 0.15)
 				)
@@
 			(effects
 				(font
-					(size 0.7 0.7)
+					(size 0.7 0.8)
 					(thickness 0.15)
 				)
@@
 			(effects
 				(font
-					(size 0.7 0.7)
+					(size 0.8 0.8)
 					(thickness 0.15)
 				)
@@
 			(effects
 				(font
-					(size 0.7 0.7)
+					(size 0.8 0.8)
 					(thickness 0.15)
 				)
@@
 			(effects
 				(font
-					(size 0.7 0.7)
+					(size 0.7 0.8)
 					(thickness 0.09)
 				)
@@
 			(effects
 				(font
-					(size 0.7 0.7)
+					(size 0.8 0.8)
 					(thickness 0.15)
 				)
@@
 			(effects
 				(font
-					(size 0.7 0.7)
+					(size 0.8 0.8)
 					(thickness 0.15)
 				)
@@
 			(effects
 				(font
-					(size 0.7 0.7)
+					(size 0.7 0.8)
 					(thickness 0.108)
 				)
@@
 			(effects
 				(font
-					(size 0.7 0.7)
+					(size 0.8 0.8)
 					(thickness 0.15)
 				)
@@
 			(effects
 				(font
-					(size 0.7 0.7)
+					(size 0.8 0.8)
 					(thickness 0.15)
 				)
@@
 			(effects
 				(font
-					(size 0.7 0.7)
+					(size 0.7 0.8)
 					(thickness 0.15)
 				)
@@
 			(effects
 				(font
-					(size 0.7 0.7)
+					(size 0.8 0.8)
 					(thickness 0.15)
 				)
@@
 			(effects
 				(font
-					(size 0.7 0.7)
+					(size 0.8 0.8)
 					(thickness 0.15)
 				)
@@
 			(effects
 				(font
-					(size 0.7 0.7)
+					(size 0.7 0.8)
 					(thickness 0.15)
 				)
@@
 			(effects
 				(font
-					(size 0.7 0.7)
+					(size 0.8 0.8)
 					(thickness 0.15)
 				)
@@
 			(effects
 				(font
-					(size 0.7 0.7)
+					(size 0.8 0.8)
 					(thickness 0.15)
 				)
@@
 			(effects
 				(font
-					(size 0.7 0.7)
+					(size 0.7 0.8)
 					(thickness 0.15)
 				)
@@
 			(effects
 				(font
-					(size 0.7 0.7)
+					(size 0.8 0.8)
 					(thickness 0.15)
 				)
@@
 			(effects
 				(font
-					(size 0.7 0.7)
+					(size 0.8 0.8)
 					(thickness 0.15)
 				)
@@
 			(effects
 				(font
-					(size 0.7 0.7)
+					(size 0.7 0.8)
 					(thickness 0.09)
 				)
@@
 			(effects
 				(font
-					(size 0.7 0.7)
+					(size 0.8 0.8)
 					(thickness 0.15)
 				)
@@
 			(effects
 				(font
-					(size 0.7 0.7)
+					(size 0.8 0.8)
 					(thickness 0.15)
 				)
@@
 			(effects
 				(font
-					(size 0.7 0.7)
+					(size 0.7 0.8)
 					(thickness 0.15)
 				)
@@
 	(footprint "Symbol:KiCad-Logo2_5mm_SilkScreen"
 		(layer "B.Cu")
-		(at 52 66 -90)
+		(at 33 71.5 -90)
 		(descr "KiCad Logo")
 		(tags "Logo KiCad")
@@
 	)
 	(gr_circle
-		(center 41.5 66.136357)
-		(end 47.72289 68.786357)
+		(center 38.25 65.15727)
+		(end 39.4 66.6)
 		(stroke
 			(width 0.1)
@@
 		)
 	)
-	(gr_text "version0.1"
-		(at 38.8 61.9 90)
+	(gr_text "v0.1"
+		(at 38.9 63.6 90)
 		(layer "B.SilkS")
 		(effects
