File: Project-4-MCU-Datalogger/Project-4-MCU-Datalogger.kicad_sch (KiCad schematic)
At the start: 25 parts, among them U1 24LC1025, U2 24LC1025, U3 DS1337S_, U4 ATMEGA328P-AU, Y1 16 MHz, Y2 32.768 KHz

Commit message: bugfix I2C's clock signal net label (rename from SCK to SCL)
Connections:
- net SCK: no longer R3.2, U1.6 (SCL), U2.6 (SCL), U3.6 (SCL), U4.28 (PC5)
- new net SCL: R3.2, U1.6 (SCL), U2.6 (SCL), U3.6 (SCL), U4.28 (PC5)
Other:
- sheet Connectors ports: added SCL; removed none
Changed lines of the file:
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@@
 		)
 	)
-	(label "SCK"
+	(label "SCL"
 		(at 52.07 60.96 180)
 		(effects
@@
 		)
 	)
-	(label "SCK"
+	(label "SCL"
 		(at 120.65 147.32 180)
 		(effects
@@
 		)
 	)
-	(label "SCK"
+	(label "SCL"
 		(at 58.42 139.7 0)
 		(effects
@@
 		)
 	)
-	(label "SCK"
+	(label "SCL"
 		(at 207.01 77.47 180)
 		(effects
@@
 		)
 	)
-	(label "SCK"
-		(at 187.96 134.62 180)
+	(label "Vcc"
+		(at 38.1 139.7 180)
 		(effects
 			(font
@@
 		)
 	)
-	(label "Vcc"
-		(at 38.1 139.7 180)
+	(label "SCK"
+		(at 187.96 152.4 180)
 		(effects
 			(font
@@
 	)
 	(label "RESET"
-		(at 187.96 154.94 180)
+		(at 187.96 157.48 180)
 		(effects
 			(font
@@
 		)
 	)
+	(label "SCL"
+		(at 187.96 134.62 180)
+		(effects
+			(font
+				(size 1.27 1.27)
+			)
+			(justify right bottom)
+		)
+	)
 	(label "SDA"
 		(at 97.79 137.16 0)
@@
 		)
 	)
-	(label "SCK"
+	(label "SCL"
 		(at 97.79 139.7 0)
 		(effects
@@
 		)
 		(pin "RESET" passive
-			(at 187.96 154.94 180)
+			(at 187.96 157.48 180)
 			(effects
 				(font
@@
 		)
 		(pin "SCK" passive
-			(at 187.96 134.62 180)
+			(at 187.96 152.4 180)
 			(effects
 				(font
@@
 			(effects
 				(font
+					(size 1.27 1.27)
+				)
+				(justify left)
+			)
+		)
+		(pin "SCL" passive
+			(at 187.96 134.62 180)
+			(effects
+				(font
